File: Hardware/USBBoard/USBBoard.kicad_sch (KiCad schematic)
At the start: 23 parts, among them J1 USB_C_Receptacle_USB2.0, J2 POWERBOARD, Q3 BC846, Q4 BC846, U4 CH340C, U4 TC4056A

Commit message: USBBoard complete
Parts:
- removed U3: ~, Package_TO_SOT_SMD:SOT-223, symbol RemotePartsLib:XC6203
- added C11: 100nF, Capacitor_SMD:C_0805_2012Metric_Pad1.18x1.45mm_HandSolder, symbol Device:C_Small
- added C11: 10uF, Capacitor_SMD:C_0805_2012Metric_Pad1.18x1.45mm_HandSolder, symbol Device:C_Small
- added C3, C4: 1uF Tantalum, Capacitor_Tantalum_SMD:CP_EIA-3216-18_Kemet-A_Pad1.58x1.35mm_HandSolder, symbol Device:C_Small
- added C6: 0.1uF, Capacitor_SMD:C_0805_2012Metric_Pad1.18x1.45mm_HandSolder, symbol Device:C_Small
- added D1: CHARGE, Diode_SMD:D_0805_2012Metric_Pad1.15x1.40mm_HandSolder, symbol Device:LED
- added D2: STBY, Diode_SMD:D_0805_2012Metric_Pad1.15x1.40mm_HandSolder, symbol Device:LED
- added Q1, Q2: BS170F, Package_TO_SOT_SMD:SOT-23, symbol Transistor_FET:BS170F
- added Q5: AO3401A, Package_TO_SOT_SMD:SOT-23, symbol Transistor_FET:AO3401A
- added Q6: 2N7002, Package_TO_SOT_SMD:SOT-23, symbol Transistor_FET:2N7002
- added R1 (x4): 1K, Resistor_SMD:R_0805_2012Metric_Pad1.20x1.40mm_HandSolder, symbol Device:R
- added R1 (x4): 12K, Resistor_SMD:R_0805_2012Metric_Pad1.20x1.40mm_HandSolder, symbol Device:R
- added R1 (x2): 10K, Resistor_SMD:R_0805_2012Metric_Pad1.20x1.40mm_HandSolder, symbol Device:R
- added R1: 100, Resistor_SMD:R_0805_2012Metric_Pad1.20x1.40mm_HandSolder, symbol Device:R
- added U2: FS8205A, Package_SO:TSSOP-8_4.4x3mm_P0.65mm, symbol ICs:FS8205A
- added U3, U7: XC6203, Package_TO_SOT_SMD:SOT-89-3, symbol ICs:XC6203
- added U6: DW01-P, Package_SO:TSOP-6_1.65x3.05mm_P0.95mm, symbol ICs:DW01-P
- C6: value 10uF -> 0.1uF
- U4: footprint (none) -> Package_SO:SOP-8_3.9x4.9mm_P1.27mm
Connections:
- net +3.3V: now also Q1.1 (G), Q2.1 (G), R1.2, R1.2, U7.3 (VOUT); no longer C6.1, U4.16 (VCC), U4.4 (V3)
- net +3.3VP: now also C4.1, U3.3 (VOUT)
- net +5V: now also U4.16 (VCC), C6.1, R1.2, R1.2, R1.2, R1.2
- net +BATT: now also C11.1, Q5.2 (S), R1.1, R1.2, U7.2 (VIN)
- net EnPower: now also R1.2
- net GND: now also C3.2, C4.2, C6.2, Q6.2 (S), R1.1, R1.1, U2.2 (S1), U2.3 (S1), U3.1 (GND), U7.1 (GND); no longer BT1.2 (-)
- net UC_RX: now also Q1.2 (S), R1.1; no longer U4.2 (TXD)
- net UC_TX: now also Q2.2 (S), R1.1; no longer U4.3 (RXD)
- net STATE_CHARGE: now reaches R1.1, U4.7 (CHARGE)
- net STATE_CHARGE: now also D1.1 (K)
- net STATE_STBY: now reaches R1.1, U4.6 (STBY)
- net STATE_STBY: now also D2.1 (K)
- new net: Q1.3 (D), R1.1, U4.2 (TXD)
- new net: Q2.3 (D), R1.1, U4.3 (RXD)
- new net: C6.1, U4.4 (V3)
- new net: D1.2 (A), R1.1
- new net: Q6.1 (G), R1.1, R1.2
- new net: Q5.1 (G), Q6.3 (D), R1.1
- new net: C3.1, Q5.3 (D), U3.2 (VIN)
- new net: R1.2, U6.2 (CS)
- new net: C11.1, R1.2, U6.5 (VCC)
- new net: D2.2 (A), R1.1
- new net: U2.5 (G2), U6.1 (OD)
- new net: U2.4 (G1), U6.3 (OC)
- new net -BATT: BT1.2 (-), C11.2, C11.2, U2.6 (S2), U2.7 (S2), U6.6 (GND)
Other:
- note added: "ESP32 Power supply. Always on, for sleep mode"
- note added: "Peripheral power supply."
- note removed: "Package klopt niet. is te groot"
- moved on the sheet: BT1, C11, C3, C4, C6, Q3, Q4, R1, U4
