File: Hardware/GamecontrollerPeripheral/GamecontrollerPeripheral.kicad_sch (KiCad schematic)
At the start: 11 parts, among them J2 UPDI, SW1 D-Up, SW2 D-Down, SW3 D-Left, SW4 D-Right, U1 ATtiny1604-SS

Commit message: GamecontrollerPeripheral progres
Parts:
- removed SW1: D-Up, symbol Switch:SW_Push
- removed SW2: D-Down, symbol Switch:SW_Push
- removed SW3: D-Left, symbol Switch:SW_Push
- removed SW4: D-Right, symbol Switch:SW_Push
- added JP1: SDA_TOP, Jumper:SolderJumper-2_P1.3mm_Open_RoundedPad1.0x1.5mm, symbol Jumper:Jumper_2_Open
- added JP2, JP4: SDA_BOT, Jumper:SolderJumper-2_P1.3mm_Open_RoundedPad1.0x1.5mm, symbol Jumper:Jumper_2_Open
- added JP3: SCL_TOP, Jumper:SolderJumper-2_P1.3mm_Open_RoundedPad1.0x1.5mm, symbol Jumper:Jumper_2_Open
- added SW1: Joystick, InputDevices:Joystick-Universal, symbol InputDevices:Joystick
- added SW6: DPad, InputDevices:D-Pad, symbol InputDevices:DPad
- H1, H2: footprint (none) -> MountingHole:MountingHole_2.2mm_M2_DIN965_Pad
Connections:
- net +3.3V: now also SW1.1 (X-A), SW1.4 (Y-A)
- net GND: now also SW1.3 (X-B), SW1.6 (Y-B), SW1.8 (SW_B), SW1.9 (Shield), SW6.5 (GND)
- net SCL: now also JP3.2 (B), JP4.2 (B); no longer Per1.6 (SCL)
- net SDA: now also JP1.2 (B), JP2.2 (B); no longer Per1.5 (SDA)
- new net: JP1.1 (A), JP4.1 (A), Per1.5 (SDA)
- new net: JP2.1 (A), JP3.1 (A), Per1.6 (SCL)

Commit message: GamecontrollerPeripheral progres
Parts:
- added D1: LED, LED_SMD:LED_0805_2012Metric_Pad1.15x1.40mm_HandSolder, symbol Device:LED
- added R2: 1K, Resistor_SMD:R_0805_2012Metric_Pad1.20x1.40mm_HandSolder, symbol Device:R
- C2: footprint (none) -> Capacitor_SMD:C_0805_2012Metric_Pad1.18x1.45mm_HandSolder
- R1: footprint (none) -> Resistor_SMD:R_0805_2012Metric_Pad1.20x1.40mm_HandSolder
Connections:
- net +3.3V: now also D1.2 (A)
- net DPad_A: now reaches SW6.1 (A)
- net DPad_A: now also U1.2 (PA4)
- net DPad_B: now reaches SW6.2 (B)
- net DPad_B: now also U1.3 (PA5)
- net DPad_C: now reaches SW6.3 (C)
- net DPad_C: now also U1.4 (PA6)
- net DPad_D: now reaches SW6.4 (D)
- net DPad_D: now also U1.5 (PA7)
- net at U1.11 (PA1): now also R2.2
- net Joystick_X: now reaches U1.12 (PA2)
- net Joystick_X: now also SW1.2 (X-C)
- net Joystick_Y: now reaches U1.13 (PA3)
- net Joystick_Y: now also SW1.5 (Y-C)
- new net: D1.1 (K), R2.1
Other:
- moved on the sheet: C2, SW6
