File: Hardware/Main/Main.kicad_sch (KiCad schematic)
At the start: 48 parts, among them J1 POWERBOARD, SW1 SW_Push, SW2 SW_Push, SW3 SW_Push, SW4 RotaryEncoder_Switch, SW5 SW_Push, U1 TFT_ST7789, U2 ESP32-WROOM-32D, U3 TCA4311a

Commit message: Mainboard routing etc
Parts:
- C1, C2, C3, C4, C6, C7: footprint (none) -> Capacitor_SMD:C_0805_2012Metric_Pad1.18x1.45mm_HandSolder
- C5: footprint (none) -> Capacitor_SMD:CP_Elec_4x5.3
- R1, R10, R11, R12, R13, R14, R15, R16, R17, R18, R19, R2, R20, R21, R3, R4, R5, R6, R7, R8, R9: footprint (none) -> Resistor_SMD:R_0805_2012Metric_Pad1.20x1.40mm_HandSolder
- U3: footprint (none) -> Package_SO:SOIC-8_3.9x4.9mm_P1.27mm
Connections:
- net +3.3V: no longer C7.1
- net +3.3VP: now also C7.1
- net BatSense: now also U2.5 (SENSOR_VN); no longer U2.4 (SENSOR_VP)
- net ChargeState: now also U2.4 (SENSOR_VP); no longer U2.5 (SENSOR_VN)

Commit message: Progress with main board
Parts:
- added J2: ProgHeader, Connectors:ESP32ProgHeader, symbol Connectors:ESP32ProgHeader
- added R22, R23, R24, R25, R26: 1K, Resistor_SMD:R_0805_2012Metric_Pad1.20x1.40mm_HandSolder, symbol Device:R
Connections:
- net +3.3V: now also J2.2 (3.3V)
- net ButtonA: now also U2.10 (IO25)
- net ButtonB: now also U2.14 (IO12)
- net GND: now also J2.4 (GND)
- net ID0Prog: now also J2.6 (ESP_IO0)
- net RESET: now also J2.1 (ESP_EN)
- net RX: now also J2.5 (ESP_RXD)
- net RotaryA: now also U2.12 (IO27)
- net RotaryB: now also U2.13 (IO14)
- net RotaryButton: now also U2.11 (IO26)
- net SCL_ESP: now also U2.8 (IO32)
- net SDA_ESP: now also U2.9 (IO33)
- net TX: now also J2.3 (ESP_TXD)
- net WS2812Led: now also U2.6 (IO34)
- net at U1.3 (SCK): now also R22.1
- net at U1.4 (SDA): now also R23.1
- net at U1.5 (RES): now also R24.1
- net at U1.6 (DC): now also R25.1
- net at U1.7 (BLK): now also R26.1
- net TFT_BLK: now reaches U2.17 (SHD/SD2)
- net TFT_BLK: now also R26.2
- net TFT_DC: now reaches U2.18 (SWP/SD3)
- net TFT_DC: now also R25.2
- net TFT_RES: now reaches U2.19 (SCS/CMD)
- net TFT_RES: now also R24.2
- net TFT_SCK: now reaches U2.20 (SCK/CLK)
- net TFT_SCK: now also R22.2
- net TFT_SDA: now reaches U2.21 (SDO/SD0)
- net TFT_SDA: now also R23.2
Other:
- moved on the sheet: C7, U1

Commit message: Mainboard r0.1
Connections:
- net GND: no longer H1.1, H2.1, H3.1, H4.1
Changed lines of the file:
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@@
-    )
-  )
-  (symbol (lib_id "power:GND") (at 108.585 127.635 0) (unit 1)
-    (in_bom yes) (on_board yes) (dnp no) (fields_autoplaced)
-    (property "Reference" "#PWR036" (at 108.585 133.985 0)
-      (effects (font (size 1.27 1.27)) hide)
-    )
-    (property "Value" "GND" (at 108.585 132.715 0)
-      (effects (font (size 1.27 1.27)))
-    )
-    (property "Footprint" "" (at 108.585 127.635 0)
-      (effects (font (size 1.27 1.27)) hide)
-    )
-    (property "Datasheet" "" (at 108.585 127.635 0)
-      (effects (font (size 1.27 1.27)) hide)
-    )
-    (pin "1")
-    (instances
-      (project "Main"
-        (path "/224a696e-f17d-43f5-99bb-b8987287a3d0"
-          (reference "#PWR036") (unit 1)
-        )
-      )
-      (project "UniversalRemote"
-        (path "/72bb8164-c3f7-4d71-82ed-b932f7d5ae7a"
-          (reference "#PWR015") (unit 1)
-        )
-      )
-      (project "USBBoard"
-        (path "/afb12ae8-e002-40c8-bda7-949acd5a5f35"
-          (reference "#PWR04") (unit 1)
-        )
-      )
     )
   )
@@
     )
   )
-  (symbol (lib_id "power:GND") (at 99.695 127.635 0) (unit 1)
-    (in_bom yes) (on_board yes) (dnp no) (fields_autoplaced)
-    (property "Reference" "#PWR035" (at 99.695 133.985 0)
-      (effects (font (size 1.27 1.27)) hide)
-    )
-    (property "Value" "GND" (at 99.695 132.715 0)
-      (effects (font (size 1.27 1.27)))
-    )
-    (property "Footprint" "" (at 99.695 127.635 0)
-      (effects (font (size 1.27 1.27)) hide)
-    )
-    (property "Datasheet" "" (at 99.695 127.635 0)
-      (effects (font (size 1.27 1.27)) hide)
-    )
-    (pin "1")
-    (instances
-      (project "Main"
-        (path "/224a696e-f17d-43f5-99bb-b8987287a3d0"
-          (reference "#PWR035") (unit 1)
-        )
-      )
-      (project "UniversalRemote"
-        (path "/72bb8164-c3f7-4d71-82ed-b932f7d5ae7a"
-          (reference "#PWR015") (unit 1)
-        )
-      )
-      (project "USBBoard"
-        (path "/afb12ae8-e002-40c8-bda7-949acd5a5f35"
-          (reference "#PWR05") (unit 1)
-        )
-      )
-    )
-  )
   (symbol (lib_id "power:GND") (at 87.63 55.245 0) (unit 1)
     (in_bom yes) (on_board yes) (dnp no) (fields_autoplaced)
@@
     )
   )
-  (symbol (lib_id "power:GND") (at 108.585 114.935 0) (unit 1)
-    (in_bom yes) (on_board yes) (dnp no) (fields_autoplaced)
-    (property "Reference" "#PWR034" (at 108.585 121.285 0)
-      (effects (font (size 1.27 1.27)) hide)
-    )
-    (property "Value" "GND" (at 108.585 120.015 0)
-      (effects (font (size 1.27 1.27)))
-    )
-    (property "Footprint" "" (at 108.585 114.935 0)
-      (effects (font (size 1.27 1.27)) hide)
-    )
-    (property "Datasheet" "" (at 108.585 114.935 0)
-      (effects (font (size 1.27 1.27)) hide)
-    )
-    (pin "1")
-    (instances
-      (project "Main"
-        (path "/224a696e-f17d-43f5-99bb-b8987287a3d0"
-          (reference "#PWR034") (unit 1)
-        )
-      )
-      (project "UniversalRemote"
-        (path "/72bb8164-c3f7-4d71-82ed-b932f7d5ae7a"
-          (reference "#PWR015") (unit 1)
-        )
-      )
-      (project "USBBoard"
-        (path "/afb12ae8-e002-40c8-bda7-949acd5a5f35"
-          (reference "#PWR04") (unit 1)
-        )
-      )
-    )
-  )
   (symbol (lib_id "power:+3.3V") (at 48.26 201.93 0) (unit 1)
     (in_bom yes) (on_board yes) (dnp no)
@@
         )
       )
-    )
-  )
-  (symbol (lib_id "power:GND") (at 99.695 114.935 0) (unit 1)
-    (in_bom yes) (on_board yes) (dnp no) (fields_autoplaced)
-    (property "Reference" "#PWR033" (at 99.695 121.285 0)
-      (effects (font (size 1.27 1.27)) hide)
-    )
-    (property "Value" "GND" (at 99.695 120.015 0)
-      (effects (font (size 1.27 1.27)))
-    )
-    (property "Footprint" "" (at 99.695 114.935 0)
-      (effects (font (size 1.27 1.27)) hide)
-    )
-    (property "Datasheet" "" (at 99.695 114.935 0)
-      (effects (font (size 1.27 1.27)) hide)
-    )
-    (pin "1")
-    (instances
-      (project "Main"
-        (path "/224a696e-f17d-43f5-99bb-b8987287a3d0"
-          (reference "#PWR033") (unit 1)
-        )
-      )
-      (project "UniversalRemote"
-        (path "/72bb8164-c3f7-4d71-82ed-b932f7d5ae7a"
-          (reference "#PWR015") (unit 1)
-        )
-      )
-      (project "USBBoard"
-        (path "/afb12ae8-e002-40c8-bda7-949acd5a5f35"
-          (reference "#PWR05") (unit 1)
-        )
-      )

Commit message: Need to make more commits; Changed design to use horizontal peripheral connectors. Changed models, more compact design. Still in progress
Parts:
- H3, H4, H5, H6: footprint MountingHole:MountingHole_2.2mm_M2_DIN965_Pad -> MountingHole:MountingHole_3.2mm_M3_DIN965_Pad
Changed lines of the file:
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@@
       (effects (font (size 1.27 1.27)) (justify left) hide)
     )
-    (property "Footprint" "MountingHole:MountingHole_2.2mm_M2_DIN965_Pad" (at 108.585 137.16 0)
+    (property "Footprint" "MountingHole:MountingHole_3.2mm_M3_DIN965_Pad" (at 108.585 137.16 0)
       (effects (font (size 1.27 1.27)) hide)
     )
@@
       (effects (font (size 1.27 1.27)) (justify left) hide)
     )
-    (property "Footprint" "MountingHole:MountingHole_2.2mm_M2_DIN965_Pad" (at 99.695 125.095 0)
+    (property "Footprint" "MountingHole:MountingHole_3.2mm_M3_DIN965_Pad" (at 99.695 125.095 0)
       (effects (font (size 1.27 1.27)) hide)
     )
@@
       (effects (font (size 1.27 1.27)) (justify left) hide)
     )
-    (property "Footprint" "MountingHole:MountingHole_2.2mm_M2_DIN965_Pad" (at 99.695 137.16 0)
+    (property "Footprint" "MountingHole:MountingHole_3.2mm_M3_DIN965_Pad" (at 99.695 137.16 0)
       (effects (font (size 1.27 1.27)) hide)
     )
@@
       (effects (font (size 1.27 1.27)) (justify left) hide)
     )
-    (property "Footprint" "MountingHole:MountingHole_2.2mm_M2_DIN965_Pad" (at 108.585 125.095 0)
-      (effects (font (size 1.27 1.27)) hide)
-    )
+    (property "Footprint" "MountingHole:MountingHole_3.2mm_M3_DIN965_Pad" (at 108.585 125.095 0)
+      (effects (font (size 1.27 1.27)) hide)
+    )

Commit message: Add extra mountingscrew to side peripherals
Parts:
- Per2: footprint Connectors:PeripheralMaster -> Connectors:PeripheralMaster_Right
- Per3: footprint Connectors:PeripheralMaster -> Connectors:PeripheralMaster_Left
Changed lines of the file:
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@@
       (effects (font (size 1.27 1.27)))
     )
-    (property "Footprint" "Connectors:PeripheralMaster" (at 81.28 71.755 0)
+    (property "Footprint" "Connectors:PeripheralMaster_Right" (at 81.28 71.755 0)
       (effects (font (size 1.27 1.27)) hide)
     )
@@
       (effects (font (size 1.27 1.27)))
     )
-    (property "Footprint" "Connectors:PeripheralMaster" (at 121.285 72.39 0)
-      (effects (font (size 1.27 1.27)) hide)
-    )
+    (property "Footprint" "Connectors:PeripheralMaster_Left" (at 121.285 72.39 0)
+      (effects (font (size 1.27 1.27)) hide)
+    )
